File: JTAG_ISP-HDR/JTAG_ISP-HDR.kicad_sch (KiCad schematic)
At the start: 6 parts, among them J1 Conn_01x08, J2 Conn_01x08

Commit message: # [SCHÉMA] + Ajout des bon noms de footprint pour les pièces SMD pour concorder avec celle du PCB. + Ajout de BOM pour les 2 PCB. * Correction de la cartouche;     * Version actuelle.
Parts:
- C1: footprint Capacitor_THT:C_Disc_D3.0mm_W2.0mm_P2.50mm -> Capacitor_SMD:C_1206_3216Metric_Pad1.33x1.80mm_HandSolder
- D1: footprint LED_THT:LED_D3.0mm -> LED_SMD:LED_1210_3225Metric_Pad1.42x2.65mm_HandSolder
- R1: footprint Resistor_THT:R_Axial_DIN0207_L6.3mm_D2.5mm_P10.16mm_Horizontal -> Resistor_SMD:R_1206_3216Metric_Pad1.30x1.75mm_HandSolder
Changed lines of the file:
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@@
     (title "JTAG_ISP / HDR")
     (date "2022-04-15")
-    (rev "v5.4.0")
+    (rev "v6.0.0")
   )
   (junction (at 127 35.179) (diameter 0) (color 0 0 0 0)
@@
     (property "Reference" "D1" (id 0) (at 93.0275 74.93 0))
     (property "Value" "LED" (id 1) (at 93.0275 77.47 0))
-    (property "Footprint" "LED_THT:LED_D3.0mm" (id 2) (at 91.44 82.296 0)
+    (property "Footprint" "LED_SMD:LED_1210_3225Metric_Pad1.42x2.65mm_HandSolder" (id 2) (at 91.44 82.296 0)
       (effects (font (size 1.27 1.27)) hide)
     )
@@
       (effects (font (size 1.27 1.27)) (justify left))
     )
-    (property "Footprint" "Resistor_THT:R_Axial_DIN0207_L6.3mm_D2.5mm_P10.16mm_Horizontal" (id 2) (at 100.33 88.392 90)
+    (property "Footprint" "Resistor_SMD:R_1206_3216Metric_Pad1.30x1.75mm_HandSolder" (id 2) (at 100.33 88.392 90)
       (effects (font (size 1.27 1.27)) hide)
     )
@@
     (property "Reference" "C1" (id 0) (at 97.155 37.084 90))
     (property "Value" "100nF" (id 1) (at 97.155 39.624 90))
-    (property "Footprint" "Capacitor_THT:C_Disc_D3.0mm_W2.0mm_P2.50mm" (id 2) (at 100.965 43.7388 0)
+    (property "Footprint" "Capacitor_SMD:C_1206_3216Metric_Pad1.33x1.80mm_HandSolder" (id 2) (at 100.965 43.7388 0)
       (effects (font (size 1.27 1.27)) hide)
     )
@@
     )
     (path "/adc24e49-3665-4c83-8bdf-87b8907ad01f"
-      (reference "C1") (unit 1) (value "100nF") (footprint "Capacitor_THT:C_Disc_D3.0mm_W2.0mm_P2.50mm")
+      (reference "C1") (unit 1) (value "100nF") (footprint "Capacitor_SMD:C_1206_3216Metric_Pad1.33x1.80mm_HandSolder")
     )
     (path "/3545dbc8-30ce-435d-acf7-b7a61060bd39"
-      (reference "D1") (unit 1) (value "LED") (footprint "LED_THT:LED_D3.0mm")
+      (reference "D1") (unit 1) (value "LED") (footprint "LED_SMD:LED_1210_3225Metric_Pad1.42x2.65mm_HandSolder")
     )
     (path "/47d80b05-190b-46ea-97e3-8322a4011f66"
@@
     )
     (path "/48b8ef63-27a0-4ab0-a935-c9d2cd80ed39"
-      (reference "R1") (unit 1) (value "100") (footprint "Resistor_THT:R_Axial_DIN0207_L6.3mm_D2.5mm_P10.16mm_Horizontal")
-    )
-  )
+      (reference "R1") (unit 1) (value "100") (footprint "Resistor_SMD:R_1206_3216Metric_Pad1.30x1.75mm_HandSolder")
+    )
+  )
